File: W1209_PIC.brd (EAGLE design)
At the start: 49 x 40 mm, 35 parts, among them IC1 MCP1700-33, IC2 PIC18F14K50SS, K1 DS1E-12V, Q1 BC817-40SMD, X1 2X381, X2 53261-05, X3 NTC, X4 2X381

Commit message: Add files via upload
Parts:
- removed X2: 53261-05, con-molex:53261-05
- added C7: 100n, resistor:C0805
- added R5: 470, resistor:R0805
- added R6: 10K, resistor:R0805
- added R7, R8, R9: 180, resistor:R0805
- added X5: MKDSN1,5/2-5,08, con-phoenix-508:MKDSN1,5/2-5,08
- C4: device resistor:SMC_C -> resistor:SMC_B
- IC1: value MCP1700-33 -> MCP1825S-33; device microchip2:SOT23 -> microchip2:SOT223
- K1: value DS1E-12V -> JJM1A-12V; device relay:DS1E -> relay:JJM1A
- R2: value 470 -> 10; device resistor:R0805 -> resistor:R2512
- R3: value 100 -> 470
- R4: value 470 -> 100
- X1: value 2X381 -> MKDSN1,5/2-5,08; device con-phoenix-3.81:1751248 -> con-phoenix-508:MKDSN1,5/2-5,08
- X4: value 2X381 -> 53047-05; device con-phoenix-3.81:1751248 -> con-molex:53047-05
- moved R4 44.1 mm to (36.6, 37.7), turned to 90 degrees
- moved X4 36.0 mm to (11.3, 35.9), turned to 270 degrees
- moved C3 33.1 mm to (40.4, 14.4), turned to 270 degrees
- moved R2 22.4 mm to (30.0, 10.0), turned to 180 degrees
- moved C5 22.2 mm to (12.4, 18.6), turned to 270 degrees
- moved SG1 18.8 mm to (38.0, 28.6), turned to 135 degrees
- moved C6 13.6 mm to (25.4, 14.4), turned to 0 degrees
- moved F2 7.00 mm to (7.77, 0.85)
- moved F1 6.00 mm to (48.3, 32.9)
- moved R3 5.26 mm to (38.9, 33.9), turned to 180 degrees
- moved D1 4.44 mm to (34.3, 14.0), turned to 180 degrees
- moved D2 2.29 mm to (7.15, 9.85)
- moved C1 1.81 mm to (2.10, 31.2), turned to 180 degrees
- moved C4 1.42 mm to (47.7, 20.3), turned to 270 degrees
- moved C2 1.41 mm to (38.4, 9.53)
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Connections:
- new net N$6: R2.1, X1.2
- new net N$7: DS1.P$12, R7.1
- new net N$8: DS1.P$8, R9.1
- new net N$9: DS1.P$9, R8.1
- net +12V: now also R2.2; no longer X1.1
- net +5V: now also IC1.3, R6.2, X4.2; no longer IC1.2, X2.2
- net AN0: now also C7.1, R6.1, X3.1; no longer X3.2
- net D+: now also R4.2, X4.5; no longer R2.2, X2.5
- net GND: now also C7.2, IC1.2, IC1.4, X1.1, X3.2, X4.1; no longer IC1.1, X1.2, X2.1, X3.1
- net K1: now also R7.2; no longer DS1.P$12
- net K2: now also R8.2; no longer DS1.P$9
- net K3: now also R9.2, X4.3; no longer DS1.P$8, X2.3
- net N$1: now also IC1.1; no longer IC1.3
- net N$11: now also R5.2; no longer R4.2
- net N$14: now also R3.1; no longer R2.1
- net N$2: now also K1.2; no longer K1.6
- net N$3: now also K1.C, X5.2; no longer K1.7, X4.1
- net N$4: now also K1.NO, X5.1; no longer K1.12, X4.2
- net N$5: now also R4.1; no longer R3.1
- net RELE: now also R5.1; no longer R4.1
- net SW3: now also X4.4; no longer X2.4
Routing:
- net SEG_D: track 33.7 -> 73.9 mm, vias 1 -> 4
- net D+: track 83.4 -> 48.5 mm, vias 4 -> 0
- net RELE: track 51.2 -> 18.1 mm
- net K2: track 0.00 -> 29.4 mm, vias 0 -> 2
- net AN0: track 40.4 -> 64.0 mm
- net +5V: track 87.1 -> 105.2 mm
- net SEG_B: track 52.0 -> 37.5 mm
- net SW2: track 46.2 -> 31.8 mm, vias 2 -> 1
- net SW3: track 73.5 -> 84.0 mm, vias 5 -> 3
- net SEG_C: track 42.5 -> 32.3 mm
- net N$6: track 0.00 -> 9.87 mm
- net SEG_G: track 42.8 -> 33.4 mm
- net N$3: track 8.12 -> 17.3 mm
- net N$9: track 0.00 -> 8.72 mm
- net N$1: track 21.1 -> 13.5 mm, vias 3 -> 0
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Other:
- board text added: "W1209_PIC (C) 2023 Dario's Automation"

Commit message: Add files via upload
Parts:
- moved C1 6.98 mm to (8.79, 33.2), turned to 270 degrees
- moved R1 5.38 mm to (8.23, 37.7), turned to 90 degrees
- moved R6 4.95 mm to (32.1, 24.4), turned to 0 degrees
- moved C5 2.90 mm to (9.64, 17.8), turned to 180 degrees
- moved JP2 1.90 mm to (15.1, 33.0)
- moved R7 1.27 mm to (18.4, 35.4)
- moved C7 1.18 mm to (41.2, 30.1)
- moved C6 1.00 mm to (24.4, 14.4)
- moved R3 1.00 mm to (39.9, 33.9)
- moved USB1 1.00 mm to (1.21, 16.5), flipped to the top, turned to 0 degrees
- moved IC2 0.93 mm to (6.30, 25.9)
- moved R8 0.90 mm to (25.4, 31.6)
- moved R9 0.90 mm to (32.4, 34.6)
- moved Q1 0.63 mm to (4.12, 9.64)
- moved R5 0.63 mm to (1.31, 9.53)
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Connections:
- net GND: now also X1.2; no longer X1.1
- net K1: now also C1.1, IC2.4, R1.1, X4.3; no longer IC2.2
- net K3: now also IC2.2; no longer C1.1, IC2.4, R1.1, X4.3
- net N$3: now also X5.1; no longer X5.2
- net N$4: now also X5.2; no longer X5.1
- net N$6: now also X1.1; no longer X1.2
Routing:
- net RELE: track 18.1 -> 86.4 mm, vias 2 -> 4
- net K2: track 29.4 -> 90.9 mm
- net D+: track 48.5 -> 96.8 mm, vias 0 -> 8
- net SEG_E: track 18.0 -> 57.6 mm, vias 1 -> 4
- net +5V: track 105.2 -> 143.7 mm, vias 2 -> 7
- net SEG_D: track 73.9 -> 49.5 mm, vias 4 -> 1
- net SEG_B: track 37.5 -> 54.8 mm, vias 1 -> 4
- net SW3: track 84.0 -> 68.5 mm, vias 3 -> 4
- net SW1: track 23.3 -> 38.8 mm
- net N$15: track 30.8 -> 44.2 mm, vias 2 -> 6
- net AN0: track 64.0 -> 52.6 mm, vias 1 -> 3
- net SW2: track 31.8 -> 22.8 mm, vias 1 -> 0
- net N$3: track 17.3 -> 10.2 mm
- net GND: track 196.9 -> 203.7 mm, vias 8 -> 7
- net K3: track 43.4 -> 38.0 mm, vias 3 -> 2
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Other:
- board text added: "12V"
- board text added: "OUT"
- board text added: "Prog"
- board text added: "TH"
