File: W1209_PIC.sch (EAGLE design)
At the start: 35 parts, among them IC1 MCP1700-33, IC2 PIC18F14K50SS, K1 DS1E-12V, Q1 BC817-40SMD, X1 2X381, X2 53261-05, X3 NTC, X4 2X381

Commit message: Add files via upload
Parts:
- removed X4: 2X381, con-phoenix-3.81:2X381
- added C7: 100n, resistor:C-EUC0805
- added R5: 470, resistor:R-EU_R0805
- added R6: 10K, resistor:R-EU_R0805
- added R7, R8, R9: 180, resistor:R-EU_R0805
- added X5: MKDSN1,5/2-5,08, con-phoenix-508:MKDSN1,5/2-5,08
- C4: device resistor:CPOL-EUSMCC -> resistor:CPOL-EUSMCB
- IC1: value MCP1700-33 -> MCP1825S-33; device microchip2:MCP1700SOT23 -> microchip2:MCP1825SSOT223
- K1: value DS1E-12V -> JJM1A-12V; device relay:DS1E-12V -> relay:JJM1A-12V
- R2: value 470 -> 10; device resistor:R-EU_R0805 -> resistor:R-EU_R2512
- R3: value 100 -> 470
- R4: value 470 -> 100
- X1: value 2X381 -> MKDSN1,5/2-5,08; device con-phoenix-3.81:2X381 -> con-phoenix-508:MKDSN1,5/2-5,08
Connections:
- new net N$6: R2.1, X1-2.KL
- new net N$7: DS1.CA@1, R7.1
- new net N$8: DS1.CA@3, R9.1
- net +12V: now also K11.1, R2.2; no longer K11.+, X1.1
- net +5V: now also R6.2
- net AN0: now also C7.1, R6.1, X3-1.S; no longer X3-2.S
- net D+: now also R4.2; no longer R2.2
- net GND: now also C7.2, X1-1.KL, X3-2.S; no longer X1.2, X3-1.S
- net K1: now also R7.2; no longer DS1.CA@1
- net K2: now also R8.1, R8.2
- net K3: now also R9.2; no longer DS1.CA@3
- net N$11: now also R5.2; no longer R4.2
- net N$14: now also R3.1; no longer R2.1
- net N$2: now also K11.2; no longer K11.-
- net N$3: now also X5-2.KL; no longer X4.1
- net N$4: now also X5-1.KL; no longer X4.2
- net N$5: now also R4.1; no longer R3.1
- net RELE: now also R5.1; no longer R4.1
Other:
- moved on the sheet: C2, D1, R2, R3, R4

Commit message: Add files via upload
Parts:
- removed X2: 53261-05, con-molex:53261-05
- added X4: 53047-05, con-molex:53047-05
Connections:
- new net N$9: DS1.CA@2, R8.1
- net +5V: now also X4-2.S; no longer X2-2.S
- net D+: now also X4-5.S; no longer X2-5.S
- net GND: now also X4-1.S; no longer X2-1.S
- net K2: no longer DS1.CA@2, R8.1
- net K3: now also X4-3.S; no longer X2-3.S
- net SW3: now also X4-4.S; no longer X2-4.S
Changed lines of the file:
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@@
 <setting verticaltext="up"/>
 </settings>
-<grid distance="0.1" unitdist="inch" unit="inch" style="lines" multiple="1" display="no" altdistance="0.05" altunitdist="inch" altunit="inch"/>
+<grid distance="0.1" unitdist="inch" unit="inch" style="lines" multiple="1" display="no" altdistance="0.01" altunitdist="inch" altunit="inch"/>
 <layers>
 <layer number="1" name="Top" color="4" fill="1" visible="no" active="no"/>
@@
 </class>
 <class number="2" name="N2" width="0.762" drill="0">
+<clearance class="2" value="0.635"/>
 </class>
 <class number="3" name="N3" width="0.4064" drill="0">
@@
 <part name="R1" library="resistor" deviceset="R-EU_" device="R0805" value="10K"/>
 <part name="C1" library="resistor" deviceset="C-EU" device="C0805" value="100n"/>
-<part name="X2" library="con-molex" deviceset="53?-05" device="261"/>
 <part name="GND1" library="supply1" deviceset="GND" device=""/>
 <part name="GND5" library="supply1" deviceset="GND" device=""/>
@@
 <part name="R8" library="resistor" deviceset="R-EU_" device="R0805" value="180"/>
 <part name="R9" library="resistor" deviceset="R-EU_" device="R0805" value="180"/>
+<part name="X4" library="con-molex" deviceset="53?-05" device="047"/>
 </parts>
 <sheets>
@@
 <instance part="R1" gate="G$1" x="7.62" y="119.38" rot="R90"/>
 <instance part="C1" gate="G$1" x="7.62" y="109.22"/>
-<instance part="X2" gate="-1" x="12.7" y="78.74" rot="MR0"/>
-<instance part="X2" gate="-2" x="12.7" y="76.2" rot="MR0"/>
-<instance part="X2" gate="-3" x="12.7" y="73.66" rot="MR0"/>
-<instance part="X2" gate="-4" x="12.7" y="71.12" rot="MR0"/>
-<instance part="X2" gate="-5" x="12.7" y="68.58" rot="MR0"/>
 <instance part="GND1" gate="1" x="7.62" y="92.71"/>
 <instance part="GND5" gate="1" x="25.4" y="59.69"/>
@@
 <instance part="R8" gate="G$1" x="149.86" y="154.94" rot="R90"/>
 <instance part="R9" gate="G$1" x="154.94" y="154.94" rot="R90"/>
+<instance part="X4" gate="-1" x="12.7" y="78.74" rot="MR0"/>
+<instance part="X4" gate="-2" x="12.7" y="76.2" rot="MR0"/>
+<instance part="X4" gate="-3" x="12.7" y="73.66" rot="MR0"/>
+<instance part="X4" gate="-4" x="12.7" y="71.12" rot="MR0"/>
+<instance part="X4" gate="-5" x="12.7" y="68.58" rot="MR0"/>
 </instances>
 <busses>
@@
 </segment>
 <segment>
-<pinref part="X2" gate="-1" pin="S"/>
 <wire x1="15.24" y1="78.74" x2="25.4" y2="78.74" width="0.1524" layer="91"/>
 <wire x1="25.4" y1="78.74" x2="25.4" y2="62.23" width="0.1524" layer="91"/>
 <pinref part="GND5" gate="1" pin="GND"/>
+<pinref part="X4" gate="-1" pin="S"/>
 </segment>
 <segment>
@@
 </segment>
 <segment>
-<pinref part="X2" gate="-2" pin="S"/>
 <pinref part="P+2" gate="1" pin="+5V"/>
 <wire x1="15.24" y1="76.2" x2="20.32" y2="76.2" width="0.1524" layer="91"/>
 <wire x1="20.32" y1="76.2" x2="20.32" y2="83.82" width="0.1524" layer="91"/>
+<pinref part="X4" gate="-2" pin="S"/>
 </segment>
 <segment>
@@
 </segment>
 <segment>
-<pinref part="X2" gate="-5" pin="S"/>
 <label x="15.24" y="68.58" size="1.778" layer="95"/>
 <wire x1="15.24" y1="68.58" x2="34.29" y2="68.58" width="0.1524" layer="91"/>
+<pinref part="X4" gate="-5" pin="S"/>
 </segment>
 <segment>
@@
 </segment>
 <segment>
-<pinref part="X2" gate="-4" pin="S"/>
 <label x="15.24" y="71.12" size="1.778" layer="95"/>
 <wire x1="15.24" y1="71.12" x2="33.02" y2="71.12" width="0.1524" layer="91"/>
+<pinref part="X4" gate="-4" pin="S"/>
 </segment>
 <segment>
@@
 <net name="K2" class="0">
 <segment>
-<pinref part="DS1" gate="G$1" pin="CA@2"/>
-<wire x1="149.86" y1="142.24" x2="149.86" y2="149.86" width="0.1524" layer="91"/>
-<pinref part="R8" gate="G$1" pin="1"/>
-</segment>
-<segment>
 <pinref part="IC2" gate="G$1" pin="RA4/OSC2"/>
 <wire x1="68.58" y1="86.36" x2="55.88" y2="86.36" width="0.1524" layer="91"/>
@@
 <net name="K3" class="0">
 <segment>
-<pinref part="X2" gate="-3" pin="S"/>
 <label x="15.24" y="73.66" size="1.778" layer="95"/>
 <wire x1="15.24" y1="73.66" x2="48.26" y2="73.66" width="0.1524" layer="91"/>
@@
 <junction x="7.62" y="111.76"/>
 <label x="58.42" y="83.82" size="1.778" layer="95"/>
+<pinref part="X4" gate="-3" pin="S"/>
 </segment>
 <segment>
@@
 </segment>
 </net>
+<net name="N$9" class="0">
+<segment>
+<pinref part="R8" gate="G$1" pin="1"/>
+<pinref part="DS1" gate="G$1" pin="CA@2"/>
+<wire x1="149.86" y1="149.86" x2="149.86" y2="142.24" width="0.1524" layer="91"/>
+</segment>
+</net>

Commit message: Add files via upload
Connections:
- net GND: now also X1-2.KL; no longer X1-1.KL
- net K1: now also C1.1, IC2.RA3/!MCLR!, R1.1, X4-3.S; no longer IC2.RA5/OSC1
- net K3: now also IC2.RA5/OSC1; no longer C1.1, IC2.RA3/!MCLR!, R1.1, X4-3.S
- net N$3: now also X5-1.KL; no longer X5-2.KL
- net N$4: now also X5-2.KL; no longer X5-1.KL
- net N$6: now also X1-1.KL; no longer X1-2.KL
Other:
- moved on the sheet: X1-1, X1-2, X5-1, X5-2
Changed lines of the file:
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@@
 </class>
 <class number="2" name="N2" width="0.762" drill="0">
-<clearance class="2" value="0.635"/>
+<clearance class="2" value="0.762"/>
 </class>
 <class number="3" name="N3" width="0.4064" drill="0">
@@
 <instance part="R6" gate="G$1" x="132.08" y="198.12" rot="R180"/>
 <instance part="P+11" gate="1" x="123.19" y="201.93"/>
-<instance part="X5" gate="-1" x="208.28" y="71.12"/>
-<instance part="X5" gate="-2" x="208.28" y="66.04"/>
-<instance part="X1" gate="-1" x="10.16" y="190.5" rot="R180"/>
-<instance part="X1" gate="-2" x="10.16" y="195.58" rot="R180"/>
+<instance part="X5" gate="-1" x="208.28" y="66.04"/>
+<instance part="X5" gate="-2" x="208.28" y="71.12"/>
+<instance part="X1" gate="-1" x="10.16" y="195.58" rot="R180"/>
+<instance part="X1" gate="-2" x="10.16" y="190.5" rot="R180"/>
 <instance part="R7" gate="G$1" x="144.78" y="154.94" rot="R90"/>
 <instance part="R8" gate="G$1" x="149.86" y="154.94" rot="R90"/>
@@
 <pinref part="GND3" gate="1" pin="GND"/>
 <wire x1="17.78" y1="190.5" x2="17.78" y2="182.88" width="0.1524" layer="91"/>
-<pinref part="X1" gate="-1" pin="KL"/>
+<pinref part="X1" gate="-2" pin="KL"/>
 <wire x1="17.78" y1="190.5" x2="12.7" y2="190.5" width="0.1524" layer="91"/>
 </segment>
@@
 <net name="K1" class="0">
 <segment>
-<pinref part="IC2" gate="G$1" pin="RA5/OSC1"/>
-<wire x1="68.58" y1="88.9" x2="55.88" y2="88.9" width="0.1524" layer="91"/>
-<label x="58.42" y="88.9" size="1.778" layer="95"/>
-</segment>
-<segment>
 <pinref part="R7" gate="G$1" pin="2"/>
 <wire x1="144.78" y1="160.02" x2="144.78" y2="167.64" width="0.1524" layer="91"/>
 <label x="144.78" y="162.56" size="1.778" layer="95" rot="R90"/>
 </segment>
-</net>
-<net name="K2" class="0">
-<segment>
-<pinref part="IC2" gate="G$1" pin="RA4/OSC2"/>
-<wire x1="68.58" y1="86.36" x2="55.88" y2="86.36" width="0.1524" layer="91"/>
-<label x="58.42" y="86.36" size="1.778" layer="95"/>
-</segment>
-<segment>
-<pinref part="R8" gate="G$1" pin="2"/>
-<wire x1="149.86" y1="160.02" x2="149.86" y2="167.64" width="0.1524" layer="91"/>
-<label x="149.86" y="162.56" size="1.778" layer="95" rot="R90"/>
-</segment>
-</net>
-<net name="K3" class="0">
 <segment>
 <label x="15.24" y="73.66" size="1.778" layer="95"/>
@@
 <pinref part="X4" gate="-3" pin="S"/>
 </segment>
+</net>
+<net name="K2" class="0">
+<segment>
+<pinref part="IC2" gate="G$1" pin="RA4/OSC2"/>
+<wire x1="68.58" y1="86.36" x2="55.88" y2="86.36" width="0.1524" layer="91"/>
+<label x="58.42" y="86.36" size="1.778" layer="95"/>
+</segment>
+<segment>
+<pinref part="R8" gate="G$1" pin="2"/>
+<wire x1="149.86" y1="160.02" x2="149.86" y2="167.64" width="0.1524" layer="91"/>
+<label x="149.86" y="162.56" size="1.778" layer="95" rot="R90"/>
+</segment>
+</net>
+<net name="K3" class="0">
 <segment>
 <pinref part="R9" gate="G$1" pin="2"/>
 <wire x1="154.94" y1="160.02" x2="154.94" y2="167.64" width="0.1524" layer="91"/>
 <label x="154.94" y="162.56" size="1.778" layer="95" rot="R90"/>
+</segment>
+<segment>
+<pinref part="IC2" gate="G$1" pin="RA5/OSC1"/>
+<wire x1="68.58" y1="88.9" x2="55.88" y2="88.9" width="0.1524" layer="91"/>
+<label x="58.42" y="88.9" size="1.778" layer="95"/>
 </segment>
 </net>
@@
 <net name="N$3" class="2">
 <segment>
-<wire x1="205.74" y1="66.04" x2="205.74" y2="48.26" width="0.1524" layer="91"/>
 <wire x1="205.74" y1="48.26" x2="215.9" y2="48.26" width="0.1524" layer="91"/>
 <wire x1="215.9" y1="48.26" x2="215.9" y2="30.48" width="0.1524" layer="91"/>
 <pinref part="K1" gate="2" pin="P"/>
 <wire x1="215.9" y1="30.48" x2="203.2" y2="30.48" width="0.1524" layer="91"/>
-<pinref part="X5" gate="-2" pin="KL"/>
+<pinref part="X5" gate="-1" pin="KL"/>
+<wire x1="205.74" y1="66.04" x2="205.74" y2="48.26" width="0.1524" layer="91"/>
 </segment>
 </net>
@@
 <wire x1="200.66" y1="40.64" x2="203.2" y2="40.64" width="0.1524" layer="91"/>
 <pinref part="K1" gate="2" pin="S"/>
-<pinref part="X5" gate="-1" pin="KL"/>
+<pinref part="X5" gate="-2" pin="KL"/>
 <wire x1="205.74" y1="71.12" x2="200.66" y2="71.12" width="0.1524" layer="91"/>
-</segment>
-</net>
-<net name="N$6" class="3">
-<segment>
-<pinref part="R2" gate="G$1" pin="1"/>
-<wire x1="17.78" y1="195.58" x2="12.7" y2="195.58" width="0.1524" layer="91"/>
-<pinref part="X1" gate="-2" pin="KL"/>
 </segment>
 </net>
@@
 </segment>
 </net>
+<net name="N$6" class="3">
+<segment>
+<pinref part="R2" gate="G$1" pin="1"/>
+<pinref part="X1" gate="-1" pin="KL"/>
+<wire x1="17.78" y1="195.58" x2="12.7" y2="195.58" width="0.1524" layer="91"/>
+</segment>
+</net>
