File: W1209_PIC.sch (EAGLE design)
At the start: 41 parts, among them IC1 MCP1825S-33, IC2 PIC18F14K50SS, K1 JJM1A-12V, Q1 BC817-40SMD, X1 MKDSN1,5/2-5,08, X3 NTC, X4 53047-05, X5 MKDSN1,5/2-5,08

Commit message: Add files via upload
Parts:
- added R10, R11: 2K2, resistor:R-EU_R0805
- DS1: value Display 3 digit 0.39 -> Display 3 digit 0.39/0.36
- R3, R5: value 470 -> 1K
Connections:
- net +5V: now also R10.2, R11.2
- net D+: now also R11.1
- net N$3: now also X5-2.KL; no longer X5-1.KL
- net N$4: now also X5-1.KL; no longer X5-2.KL
- net SW1: now also R10.1, USB1.2
- net SW3: no longer USB1.2
Other:
- note added: "(invertire 11 con 19!! usb solo input e poi 19 con 18)"
- note added: "AN3 in effetti"
- note added: "ERRORE PCB 2023, sw3 al posto di sw1/D-"
- note added: "SERVE quarzo x USB, oppure usare PIC16F1459, identico!"
- note added: "mancano i pullup.. su pin USB..."
- note removed: "invertire 11 con 19!! usb solo input e poi 19 con 18"
- moved on the sheet: X5-2
Changed lines of the file:
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@@
 <part name="GND10" library="supply1" deviceset="GND" device=""/>
 <part name="C3" library="resistor" deviceset="C-EU" device="C0805" value="100n"/>
-<part name="R3" library="resistor" deviceset="R-EU_" device="R0805" value="470"/>
+<part name="R3" library="resistor" deviceset="R-EU_" device="R0805" value="1K"/>
 <part name="GND9" library="supply1" deviceset="GND" device=""/>
 <part name="R4" library="resistor" deviceset="R-EU_" device="R0805" value="100"/>
@@
 <part name="GND18" library="supply1" deviceset="GND" device=""/>
 <part name="Q1" library="transistor-npn" deviceset="BC817*" device="SMD" technology="-40"/>
-<part name="R5" library="resistor" deviceset="R-EU_" device="R0805" value="470"/>
+<part name="R5" library="resistor" deviceset="R-EU_" device="R0805" value="1K"/>
 <part name="S2" library="switch-omron" deviceset="10-XX" device="" value="pulsante"/>
 <part name="GND6" library="supply1" deviceset="GND" device=""/>
@@
 <part name="JP2" library="pinhead" deviceset="PINHD-1X4" device="" value="OLED left"/>
 <part name="JP1" library="pinhead" deviceset="PINHD-1X4" device="" value="OLED top"/>
-<part name="DS1" library="kingbright" deviceset="KLT36XX" device="" value="Display 3 digit 0.39"/>
+<part name="DS1" library="kingbright" deviceset="KLT36XX" device="" value="Display 3 digit 0.39/0.36"/>
 <part name="GND13" library="supply1" deviceset="GND" device=""/>
 <part name="P+5" library="supply1" deviceset="+5V" device=""/>
@@
 <part name="R9" library="resistor" deviceset="R-EU_" device="R0805" value="180"/>
 <part name="X4" library="con-molex" deviceset="53?-05" device="047"/>
+<part name="P+12" library="supply1" deviceset="+5V" device=""/>
+<part name="R10" library="resistor" deviceset="R-EU_" device="R0805" value="2K2"/>
+<part name="R11" library="resistor" deviceset="R-EU_" device="R0805" value="2K2"/>
 </parts>
 <sheets>
@@
 <text x="127" y="226.06" size="1.778" layer="91">mettere OLED I2C
 https://it.aliexpress.com/item/1-pz-0-91-pollice-OLED-modulo-0-91-bianco-blu-OLED-128X32-OLED-Display-LCD/32672229793.html</text>
-<text x="99.06" y="99.06" size="1.778" layer="91">invertire 11 con 19!! usb solo input
-e poi 19 con 18</text>
+<text x="99.06" y="99.06" size="1.778" layer="91">(invertire 11 con 19!! usb solo input
+e poi 19 con 18)</text>
+<text x="30.48" y="144.78" size="1.778" layer="91">ERRORE PCB 2023, sw3 al posto di sw1/D-</text>
+<text x="53.34" y="109.22" size="1.778" layer="91">SERVE quarzo x USB, oppure usare PIC16F1459, identico!</text>
+<text x="27.94" y="43.18" size="1.778" layer="91">mancano i pullup.. su pin USB...</text>
+<text x="53.34" y="104.14" size="1.778" layer="91">AN3 in effetti</text>
 </plain>
 <instances>
@@
 <instance part="P+11" gate="1" x="123.19" y="201.93"/>
 <instance part="X5" gate="-1" x="208.28" y="66.04"/>
-<instance part="X5" gate="-2" x="208.28" y="71.12"/>
+<instance part="X5" gate="-2" x="208.28" y="60.96"/>
 <instance part="X1" gate="-1" x="10.16" y="195.58" rot="R180"/>
 <instance part="X1" gate="-2" x="10.16" y="190.5" rot="R180"/>
@@
 <instance part="X4" gate="-4" x="12.7" y="71.12" rot="MR0"/>
 <instance part="X4" gate="-5" x="12.7" y="68.58" rot="MR0"/>
+<instance part="P+12" gate="1" x="2.54" y="55.88"/>
+<instance part="R10" gate="G$1" x="2.54" y="45.72" rot="R90"/>
+<instance part="R11" gate="G$1" x="20.32" y="45.72" rot="R90"/>
 </instances>
 <busses>
@@
 <wire x1="123.19" y1="198.12" x2="123.19" y2="199.39" width="0.1524" layer="91"/>
 </segment>
+<segment>
+<pinref part="P+12" gate="1" pin="+5V"/>
+<pinref part="R10" gate="G$1" pin="2"/>
+<wire x1="2.54" y1="53.34" x2="2.54" y2="50.8" width="0.1524" layer="91"/>
+<pinref part="R11" gate="G$1" pin="2"/>
+<wire x1="2.54" y1="50.8" x2="20.32" y2="50.8" width="0.1524" layer="91"/>
+<junction x="2.54" y="50.8"/>
+</segment>
 </net>
 <net name="N$5" class="0">
@@
 <pinref part="S2" gate="1" pin="P1"/>
 <wire x1="25.4" y1="25.4" x2="27.94" y2="25.4" width="0.1524" layer="91"/>
-<wire x1="25.4" y1="25.4" x2="25.4" y2="38.1" width="0.1524" layer="91"/>
+<wire x1="25.4" y1="25.4" x2="25.4" y2="40.64" width="0.1524" layer="91"/>
 <junction x="25.4" y="25.4"/>
 <label x="25.4" y="30.48" size="1.778" layer="95" rot="R90"/>
+<pinref part="R11" gate="G$1" pin="1"/>
+<wire x1="20.32" y1="40.64" x2="25.4" y2="40.64" width="0.1524" layer="91"/>
 </segment>
 </net>
 <net name="SW1" class="0">
 <segment>
-<wire x1="7.62" y1="25.4" x2="7.62" y2="38.1" width="0.1524" layer="91"/>
+<wire x1="7.62" y1="25.4" x2="7.62" y2="40.64" width="0.1524" layer="91"/>
 <pinref part="S1" gate="1" pin="P"/>
 <wire x1="7.62" y1="25.4" x2="10.16" y2="25.4" width="0.1524" layer="91"/>
@@
 <junction x="7.62" y="25.4"/>
 <label x="7.62" y="30.48" size="1.778" layer="95" rot="R90"/>
+<pinref part="R10" gate="G$1" pin="1"/>
+<wire x1="2.54" y1="40.64" x2="7.62" y2="40.64" width="0.1524" layer="91"/>
 </segment>
 <segment>
@@
 <wire x1="15.24" y1="71.12" x2="33.02" y2="71.12" width="0.1524" layer="91"/>
 <pinref part="X4" gate="-4" pin="S"/>
+</segment>
+<segment>
+<wire x1="15.24" y1="152.4" x2="25.4" y2="152.4" width="0.1524" layer="91"/>
+<label x="17.78" y="152.4" size="1.778" layer="95"/>
+<pinref part="USB1" gate="G$1" pin="2"/>
 </segment>
 </net>
@@
 <junction x="43.18" y="25.4"/>
 <label x="43.18" y="30.48" size="1.778" layer="95" rot="R90"/>
-</segment>
-<segment>
-<wire x1="15.24" y1="152.4" x2="25.4" y2="152.4" width="0.1524" layer="91"/>
-<label x="17.78" y="152.4" size="1.778" layer="95"/>
-<pinref part="USB1" gate="G$1" pin="2"/>
 </segment>
 <segment>
@@
 <pinref part="K1" gate="2" pin="P"/>
 <wire x1="215.9" y1="30.48" x2="203.2" y2="30.48" width="0.1524" layer="91"/>
-<pinref part="X5" gate="-1" pin="KL"/>
-<wire x1="205.74" y1="66.04" x2="205.74" y2="48.26" width="0.1524" layer="91"/>
+<pinref part="X5" gate="-2" pin="KL"/>
+<wire x1="205.74" y1="60.96" x2="205.74" y2="48.26" width="0.1524" layer="91"/>
 </segment>
 </net>
 <net name="N$4" class="2">
 <segment>
-<wire x1="200.66" y1="71.12" x2="200.66" y2="40.64" width="0.1524" layer="91"/>
+<wire x1="200.66" y1="66.04" x2="200.66" y2="40.64" width="0.1524" layer="91"/>
 <wire x1="200.66" y1="40.64" x2="203.2" y2="40.64" width="0.1524" layer="91"/>
 <pinref part="K1" gate="2" pin="S"/>
-<pinref part="X5" gate="-2" pin="KL"/>
-<wire x1="205.74" y1="71.12" x2="200.66" y2="71.12" width="0.1524" layer="91"/>
-</segment>
-</net>
+<pinref part="X5" gate="-1" pin="KL"/>
+<wire x1="205.74" y1="66.04" x2="200.66" y2="66.04" width="0.1524" layer="91"/>
+</segment>
+</net>
